File: PCB/DIAG_MULTEC.kicad_sch (KiCad schematic)
At the start: 31 parts, among them J1 CAR, J2 PC, U1 6N137, U2 LM78L05_SO8, U3 74AHC1G00, U4 MAX232

Commit message: PCB update to final components values
Parts:
- C1: value 100u -> 22u/35V
- C3: value 10u -> 10u/6V3
- D1: value MRA4007T3G -> S1M
- D2: value PWR -> PWR_GREEN
- D3: value RX -> RX_BLUE
- R3: value 3k9 -> 2k2
- R4: value 2k2 -> 4k7
- R5: value 2k2 -> 3k9
Other:
- moved on the sheet: C1, C5, D1
